Commit message: fix: update link inertial parameters

File: resources/robots/agibot_a2/urdf/agibot_a2_dof12.urdf (robot description, URDF)
Before this commit: robot a2_t2d0_ultra, 49 links, 48 joints
Links:
- link base_link: mass 18.89945962 -> 20.4197
- link head_link01: mass 1.39889495 -> 1.4191
- link head_link02: mass 0.65606942 -> 0.9109
- link left_arm_link01: mass 0.276944 -> 0.2791
- link left_arm_link02: mass 2.852114 -> 2.8105
- link left_arm_link03: mass 1.310295 -> 1.3510
- link left_arm_link04: mass 0.677343 -> 0.68884
- link left_arm_link05: mass 0.260886 -> 0.7298
- link left_arm_link06: mass 0.02504627 -> 0.0264
- link left_arm_link07: mass 0.05050219 -> 0.0229
- link left_hip_pitch: mass 5.92461880 -> 6.2946
- link left_hip_roll: mass 2.39059365 -> 2.3646
- link left_hip_yaw: mass 3.79911511 -> 3.7387
- link left_tarsus: mass 3.02166726 -> 3.3145
- link left_toe_pitch: mass 0.08772028 -> 0.0699
- link left_toe_roll: mass 1.21058213 -> 1.2068
- link right_arm_link01: mass 0.276944 -> 0.2791
- link right_arm_link02: mass 2.852114 -> 2.8300
- link right_arm_link03: mass 1.310295 -> 1.2968
- link right_arm_link04: mass 0.677343 -> 0.6888
- link right_arm_link05: mass 0.260886 -> 0.7269
- link right_arm_link06: mass 0.02504627 -> 0.0264
- link right_arm_link07: mass 0.05050219 -> 0.0229
- link right_hip_pitch: mass 5.92461880 -> 6.2850
- link right_hip_roll: mass 2.39059365 -> 2.3646
- link right_hip_yaw: mass 3.79911511 -> 3.7387
- link right_tarsus: mass 3.02166726 -> 3.3127
- link right_toe_pitch: mass 0.08772028 -> 0.0699
- link right_toe_roll: mass 1.21058213 -> 1.2068
